File: src/polaris-imu-pcb.kicad_pcb (KiCad board)
At the start: 2 copper layers, 52.5 x 80 mm, 20 parts, among them J1 GNSS, J2 RUDDER, U1 MTi-3-5A-T

Commit message: Reorganize
Parts:
- added S2: Logo, GS_Virtual:UBC_Sailbot_Logo_Plain, B.Cu at (58.5, 64.8)

Commit message: Add board characteristics
Parts:
- moved FB1 7.50 mm to (29.4, 44.7)
- moved A1 7.50 mm to (50.0, 71.0)
- moved C1 7.50 mm to (36.8, 84.9)
- moved C2 7.50 mm to (36.8, 95.1)
- moved C3 7.50 mm to (28.2, 46.9)
- moved C4 7.50 mm to (30.7, 46.9)
- moved C5 7.50 mm to (39.7, 41.0)
- moved C6 7.50 mm to (36.2, 35.8)
- moved C7 7.50 mm to (34.0, 95.1)
- moved C8 7.50 mm to (63.2, 95.1)
- moved C9 7.50 mm to (63.8, 35.8)
- moved H1 7.50 mm to (37.5, 30.8)
- moved H2 7.50 mm to (37.5, 100.8)
- moved H3 7.50 mm to (62.5, 100.8)
- moved H4 7.50 mm to (62.5, 30.8)
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