File: src/polaris-imu-pcb.kicad_pcb (KiCad board)
At the start: 2 copper layers, 52.5 x 80 mm, 21 parts, among them J1 GNSS, J2 RUDDER, U1 MTi-3-5A-T

Commit message: Small updates for rev0
Parts:
- S2: footprint GS_Virtual:UBC_Sailbot_Logo_Plain -> GS_Virtual:UBC_Sailbot_Logo_Huge
- moved S2 3.25 mm to (51.0, 61.5)
- moved S1 0.27 mm to (26.9, 73.5)
Routing:
- net /GND: vias 0 -> 42
