File: src/polaris-imu-pcb.kicad_sch (KiCad schematic)
At the start: 13 parts, among them J1 GNSS, J2 RUDDER

Commit message: Reorganize
Parts:
- added S2: Logo, GS_Virtual:UBC_Sailbot_Logo_Plain, symbol GS_Virtual:UBC_Sailbot_Logo
Other:
- moved on the sheet: S1
Changed lines of the file:
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@@
+	)
+	(symbol
+		(lib_id "GS_Virtual:UBC_Sailbot_Logo")
+		(at 44.45 105.41 0)
+		(unit 1)
+		(body_style 1)
+		(exclude_from_sim no)
+		(in_bom no)
+		(on_board yes)
+		(in_pos_files yes)
+		(dnp no)
+		(fields_autoplaced yes)
+		(property "Reference" "S2"
+			(at 44.45 101.6 0)
+			(show_name no)
+			(do_not_autoplace no)
+			(effects
+				(font
+					(size 1.27 1.27)
+				)
+			)
+		)
+		(property "Value" "Logo"
+			(at 44.45 97.028 0)
+			(hide yes)
+			(show_name no)
+			(do_not_autoplace no)
+			(effects
+				(font
+					(size 1.27 1.27)
+				)
+			)
+		)
+		(property "Footprint" "GS_Virtual:UBC_Sailbot_Logo_Plain"
+			(at 44.45 105.41 0)
+			(hide yes)
+			(show_name no)
+			(do_not_autoplace no)
+			(effects
+				(font
+					(size 1.27 1.27)
+				)
+			)
+		)
+		(property "Datasheet" ""
+			(at 44.45 105.41 0)
+			(hide yes)
+			(show_name no)
+			(do_not_autoplace no)
+			(effects
+				(font
+					(size 1.27 1.27)
+				)
+			)
+		)
+		(property "Description" "UBC Sailbot Logo"
+			(at 44.45 99.314 0)
+			(hide yes)
+			(show_name no)
+			(do_not_autoplace no)
+			(effects
+				(font
+					(size 1.27 1.27)
+				)
+			)
+		)
+		(property "SPICE Warning Override" "Virtual Part"
+			(at 44.45 105.41 0)
+			(hide yes)
+			(show_name no)
+			(do_not_autoplace no)
+			(effects
+				(font
+					(size 1.27 1.27)
+				)
+			)
+		)
+		(instances
+			(project "polaris-imu-pcb"
+				(path "/0ced2fb0-b5fd-4752-8bb9-7a03747afc00"
+					(reference "S2")
+					(unit 1)
+				)
+			)
+		)
 	)
 	(symbol
@@
 	(symbol
 		(lib_id "GS_Virtual:UBC_Sailbot_Logo")
-		(at 64.77 104.14 0)
+		(at 27.94 105.41 0)
 		(unit 1)
 		(body_style 1)
@@
 		(fields_autoplaced yes)
 		(property "Reference" "S1"
-			(at 64.77 100.33 0)
+			(at 27.94 101.6 0)
 			(show_name no)
 			(do_not_autoplace no)
@@
 		)
 		(property "Value" "Logo"
-			(at 64.77 95.758 0)
+			(at 27.94 97.028 0)
 			(hide yes)
 			(show_name no)
@@
 		)
 		(property "Footprint" "GS_Virtual:UBC_Sailbot_Logo_Silk"
-			(at 64.77 104.14 0)
+			(at 27.94 105.41 0)
 			(hide yes)
 			(show_name no)
@@
 		)
 		(property "Datasheet" ""
-			(at 64.77 104.14 0)
+			(at 27.94 105.41 0)
 			(hide yes)
 			(show_name no)
@@
 		)
 		(property "Description" "UBC Sailbot Logo"
-			(at 64.77 98.044 0)
+			(at 27.94 99.314 0)
 			(hide yes)
 			(show_name no)
@@
 		)
 		(property "SPICE Warning Override" "Virtual Part"
-			(at 64.77 104.14 0)
-			(hide yes)
-			(show_name no)
+			(at 27.94 105.41 0)
+			(hide yes)
+			(show_name no)

Commit message: Small updates for rev0
Parts:
- S2: footprint GS_Virtual:UBC_Sailbot_Logo_Plain -> GS_Virtual:UBC_Sailbot_Logo_Huge
Changed lines of the file:
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@@
 			)
 		)
-		(property "Footprint" "GS_Virtual:UBC_Sailbot_Logo_Plain"
+		(property "Footprint" "GS_Virtual:UBC_Sailbot_Logo_Huge"
 			(at 44.45 105.41 0)
 			(hide yes)
